File: RPi Arcade Hat V0-3.kicad_pcb (KiCad board)
At the start: 2 copper layers, 193.5 x 82.1 mm, 75 parts, among them J1 Raspberry_Pi_2_3, J10 Coin/Note Input, J11 +24V IN, J12 +12V OUT, J13 Player 1, J14 Player 2, J15 Player 3, J16 Player 4, J17 ICSP, J18 Program MCU, J19 Graphics LCD, J2 Player 1, J20 Channel 4, J21 Channel 3, J22 Channel 2, J23 Channel 1, J24 CCard Input, J3 Player 2, J4 Spares, J5 Player 3, J6 Player 4, J7 +24V OUT, J8 Neo Pixel Data, J9 Note Acceptor, Q16 BC847, Q4 BC847, Q5 BC847, Q6 BC847, Q7 BC847, U1 ATmega328P-A, U2 SN74HC04N, U3 LM2595S-12, Y1 16MHz Crystal

Commit message: Added Arduino Code
Parts:
- J18: value Program MCU -> Serial Program; footprint Connector_PinHeader_2.54mm:PinHeader_1x05_P2.54mm_Vertical -> Connector_PinHeader_2.54mm:PinHeader_1x06_P2.54mm_Vertical
- moved J18 10.3 mm to (209.1, 98.6), turned to 90 degrees
- moved R1 2.29 mm to (200.1, 93.2)
- moved C1 1.68 mm to (203.0, 95.6), turned to 0 degrees
Connections:
- C1 pad 1: Net-(C1-Pad1) -> RESET
- J17 pad 5: DTR -> RESET
- J18 pad 1: +5V -> DTR
- J18 pad 2: DTR -> RX
- J18 pad 4: RX -> +5V
- J18 pad 5: GND -> unconnected-(J18-Pin_5-Pad5)
- R1 pad 1: DTR -> RESET
- U1 pad 29: Net-(C1-Pad1) -> RESET
Routing:
- net RESET: track 0.00 -> 72.9 mm, vias 0 -> 2
- net Net-(C1-Pad1): track 52.0 -> 0.00 mm, vias 2 -> 0
- net DTR: track 20.1 -> 5.86 mm
- net +5V: track 44.1 -> 40.9 mm, vias 8 -> 9

Commit message: Changes made after testing
Parts:
- removed D1, D2, D3, D4: 1N4448W, Diode_SMD:D_SOD-123
- removed R9: 12k, Resistor_SMD:R_1206_3216Metric
- moved R8 2.08 mm to (192.8, 86.2)
- moved R13 2.03 mm to (150.5, 78.1)
- moved C9 2.03 mm to (150.5, 80.6)
- moved R50 1.98 mm to (192.8, 88.8)
- moved R6 1.37 mm to (150.5, 108.2), turned to 180 degrees
- moved R5 1.27 mm to (150.4, 91.9), turned to 180 degrees
- moved R7 1.22 mm to (150.3, 124.3), turned to 180 degrees
- moved C6 1.22 mm to (150.3, 129.1)
- moved R10 1.22 mm to (150.3, 126.7)
- moved C7 1.12 mm to (150.5, 113.0)
- moved R12 1.12 mm to (150.4, 94.4)
- moved R11 1.12 mm to (150.5, 110.5)
- moved C8 1.07 mm to (150.4, 96.9)
- moved R4 0.41 mm to (150.5, 75.6), turned to 180 degrees
Connections:
- R4 pad 1: Net-(D4-A) -> P4CRDBUTT
- R5 pad 1: Net-(D3-A) -> P3CRDBUTT
- R51 pad 2: Net-(R51-Pad2) -> MECH (12V)
- R6 pad 1: Net-(D2-A) -> P2CRDBUTT
- R7 pad 1: Net-(D1-A) -> P1CRDBUTT
- R8 pad 2: Net-(R51-Pad2) -> MECH (12V)
- Y1 pad 2: unconnected-(Y1-Pad2) -> GND
- Y1 pad 4: unconnected-(Y1-Pad4) -> GND
Routing:
- net +5V: track 40.9 -> 51.9 mm
- net MECH (12V): track 60.2 -> 66.7 mm
- net Net-(R51-Pad2): track 4.72 -> 0.00 mm
- net MECH (5V): track 36.2 -> 31.8 mm
- net P3CRDBUTT: track 33.4 -> 29.8 mm
- net Net-(D2-A): track 2.52 -> 0.00 mm
- net Net-(D1-A): track 2.52 -> 0.00 mm
- net Net-(D4-A): track 2.50 -> 0.00 mm
- net Net-(D3-A): track 2.47 -> 0.00 mm
- net P2CRDBUTT: track 46.1 -> 44.8 mm
- net P1CRDBUTT: track 55.3 -> 54.2 mm
- net Net-(J16-Pin_2): track 5.17 -> 4.28 mm
- net P4CRDBUTT: track 27.8 -> 28.5 mm
- net Net-(J13-Pin_2): track 4.58 -> 4.08 mm

Commit message: Fixed Input Matrix
Parts:
- added D1: 1N4448W, Diode_SMD:D_SOD-123, F.Cu at (91.2, 123.7)
- added D10: 1N4448W, Diode_SMD:D_SOD-123, F.Cu at (91.1, 107.7)
- added D11: 1N4448W, Diode_SMD:D_SOD-123, F.Cu at (96.1, 107.7)
- added D12: 1N4448W, Diode_SMD:D_SOD-123, F.Cu at (101.2, 107.7)
- added D13: 1N4448W, Diode_SMD:D_SOD-123, F.Cu at (106.1, 107.7)
- added D14: 1N4448W, Diode_SMD:D_SOD-123, F.Cu at (111.2, 107.7)
- added D15: 1N4448W, Diode_SMD:D_SOD-123, F.Cu at (116.1, 107.7)
- added D16: 1N4448W, Diode_SMD:D_SOD-123, F.Cu at (121.1, 107.7)
- added D17: 1N4448W, Diode_SMD:D_SOD-123, F.Cu at (126.1, 107.7)
- added D18: 1N4448W, Diode_SMD:D_SOD-123, F.Cu at (91.2, 91.5)
- added D19: 1N4448W, Diode_SMD:D_SOD-123, F.Cu at (96.2, 91.5)
- added D2: 1N4448W, Diode_SMD:D_SOD-123, F.Cu at (96.2, 123.7)
- added D20: 1N4448W, Diode_SMD:D_SOD-123, F.Cu at (101.1, 91.5)
- added D21: 1N4448W, Diode_SMD:D_SOD-123, F.Cu at (106.1, 91.5)
- added D22: 1N4448W, Diode_SMD:D_SOD-123, F.Cu at (111.2, 91.5)
- added D23: 1N4448W, Diode_SMD:D_SOD-123, F.Cu at (116.2, 91.5)
- added D24: 1N4448W, Diode_SMD:D_SOD-123, F.Cu at (121.1, 91.5)
- added D25: 1N4448W, Diode_SMD:D_SOD-123, F.Cu at (126.1, 91.5)
- added D26: 1N4448W, Diode_SMD:D_SOD-123, F.Cu at (91.1, 75.3)
- added D27: 1N4448W, Diode_SMD:D_SOD-123, F.Cu at (96.2, 75.3)
- added D28: 1N4448W, Diode_SMD:D_SOD-123, F.Cu at (101.2, 75.3)
- added D29: 1N4448W, Diode_SMD:D_SOD-123, F.Cu at (106.1, 75.3)
- added D3: 1N4448W, Diode_SMD:D_SOD-123, F.Cu at (101.1, 123.7)
- added D30: 1N4448W, Diode_SMD:D_SOD-123, F.Cu at (111.2, 75.3)
- added D31: 1N4448W, Diode_SMD:D_SOD-123, F.Cu at (116.2, 75.3)
- added D32: 1N4448W, Diode_SMD:D_SOD-123, F.Cu at (121.1, 75.3)
- added D33: 1N4448W, Diode_SMD:D_SOD-123, F.Cu at (126.1, 75.3)
- added D34: 1N4448W, Diode_SMD:D_SOD-123, F.Cu at (91.2, 64.9)
- added D35: 1N4448W, Diode_SMD:D_SOD-123, F.Cu at (96.2, 64.9)
- added D36: 1N4448W, Diode_SMD:D_SOD-123, F.Cu at (101.1, 64.9)
- added D37: 1N4448W, Diode_SMD:D_SOD-123, F.Cu at (106.2, 64.9)
- added D38: 1N4448W, Diode_SMD:D_SOD-123, F.Cu at (111.2, 64.9)
- added D39: 1N4448W, Diode_SMD:D_SOD-123, F.Cu at (116.2, 64.9)
- added D4: 1N4448W, Diode_SMD:D_SOD-123, F.Cu at (106.2, 123.7)
- added D40: 1N4448W, Diode_SMD:D_SOD-123, F.Cu at (121.1, 64.9)
- added D41: 1N4448W, Diode_SMD:D_SOD-123, F.Cu at (126.1, 64.9)
- added D6: 1N4448W, Diode_SMD:D_SOD-123, F.Cu at (111.3, 123.7)
- added D7: 1N4448W, Diode_SMD:D_SOD-123, F.Cu at (116.1, 123.7)
- added D8: 1N4448W, Diode_SMD:D_SOD-123, F.Cu at (121.1, 123.7)
- added D9: 1N4448W, Diode_SMD:D_SOD-123, F.Cu at (126.2, 123.7)
- C6, C7, C8, C9: value 100nF -> 300nF
- moved LED1 2.74 mm to (207.1, 87.2)
- moved R2 2.74 mm to (204.4, 87.5)
Connections:
- J2 pad 1: Column 1 -> Net-(D1-K)
- J2 pad 2: Column 2 -> Net-(D2-K)
- J2 pad 3: Column 3 -> Net-(D3-K)
- J2 pad 4: Column 4 -> Net-(D4-K)
- J2 pad 5: Column 5 -> Net-(D6-K)
- J2 pad 6: Column 6 -> Net-(D7-K)
- J2 pad 7: Column 7 -> Net-(D8-K)
- J2 pad 8: Column 8 -> Net-(D9-K)
- J3 pad 1: Column 1 -> Net-(D10-K)
- J3 pad 2: Column 2 -> Net-(D11-K)
- J3 pad 3: Column 3 -> Net-(D12-K)
- J3 pad 4: Column 4 -> Net-(D13-K)
- J3 pad 5: Column 5 -> Net-(D14-K)
- J3 pad 6: Column 6 -> Net-(D15-K)
- J3 pad 7: Column 7 -> Net-(D16-K)
- J3 pad 8: Column 8 -> Net-(D17-K)
- J4 pad 1: Column 1 -> Net-(D34-K)
- J4 pad 2: Column 2 -> Net-(D35-K)
- J4 pad 3: Column 3 -> Net-(D36-K)
- J4 pad 4: Column 4 -> Net-(D37-K)
- J4 pad 5: Column 5 -> Net-(D38-K)
- J4 pad 6: Column 6 -> Net-(D39-K)
- J4 pad 7: Column 7 -> Net-(D40-K)
- J4 pad 8: Column 8 -> Net-(D41-K)
- J5 pad 1: Column 1 -> Net-(D18-K)
- J5 pad 2: Column 2 -> Net-(D19-K)
- J5 pad 3: Column 3 -> Net-(D20-K)
- J5 pad 4: Column 4 -> Net-(D21-K)
- J5 pad 5: Column 5 -> Net-(D22-K)
- J5 pad 6: Column 6 -> Net-(D23-K)
- J5 pad 7: Column 7 -> Net-(D24-K)
- J5 pad 8: Column 8 -> Net-(D25-K)
- J6 pad 1: Column 1 -> Net-(D26-K)
- J6 pad 2: Column 2 -> Net-(D27-K)
- J6 pad 3: Column 3 -> Net-(D28-K)
- J6 pad 4: Column 4 -> Net-(D29-K)
- J6 pad 5: Column 5 -> Net-(D30-K)
- J6 pad 6: Column 6 -> Net-(D31-K)
- J6 pad 7: Column 7 -> Net-(D32-K)
- J6 pad 8: Column 8 -> Net-(D33-K)
Routing:
- net Column 1: track 263.4 -> 258.5 mm
- net Column 8: track 196.8 -> 192.2 mm
- net Column 7: track 205.5 -> 200.9 mm
- net Column 6: track 216.2 -> 211.8 mm
- net Column 5: track 224.6 -> 220.2 mm
- net Column 2: track 252.4 -> 248.1 mm
- net Column 3: track 241.6 -> 237.3 mm
- net Column 4: track 233.0 -> 228.8 mm
- net Net-(D11-K): track 0.00 -> 3.77 mm
- net Net-(D10-K): track 0.00 -> 3.76 mm
- net Net-(D12-K): track 0.00 -> 3.71 mm
- net Net-(D33-K): track 0.00 -> 3.71 mm
- net Net-(D25-K): track 0.00 -> 3.71 mm
- net Net-(D21-K): track 0.00 -> 3.71 mm
- net Net-(D16-K): track 0.00 -> 3.70 mm
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