File: RPi Arcade Hat V0-3.kicad_sch (KiCad schematic)
At the start: 75 parts, among them J1 Raspberry_Pi_2_3, J10 Coin/Note Input, J11 +24V IN, J12 +12V OUT, J13 Player 1, J14 Player 2, J15 Player 3, J16 Player 4, J17 ICSP, J18 Program MCU, J19 Graphics LCD, J2 Player 1, J20 Channel 4, J21 Channel 3, J22 Channel 2, J23 Channel 1, J24 CCard Input, J3 Player 2, J4 Spares, J5 Player 3, J6 Player 4, J7 +24V OUT, J8 Neo Pixel Data, J9 Note Acceptor, Q16 BC847, Q4 BC847, Q5 BC847, Q6 BC847, Q7 BC847, U1 ATmega328P-A, U2 SN74HC04N, U3 LM2595S-12, Y1 16MHz Crystal

Commit message: Added Arduino Code
Parts:
- removed J18: Program MCU, Connector_PinHeader_2.54mm:PinHeader_1x05_P2.54mm_Vertical, symbol Connector:Conn_01x05_Male
- added J18: Serial Program, Connector_PinHeader_2.54mm:PinHeader_1x06_P2.54mm_Vertical, symbol Connector:Conn_01x06_Pin
Connections:
- net +5V: now also J18.4 (Pin_4)
- net DTR: now also J18.1 (Pin_1); no longer J17.5 (Pin_5), R1.1
- net GND: now also J18.6 (Pin_6)
- net RX: now also J18.2 (Pin_2)
- net TX: now also J18.3 (Pin_3)
- net RESET: now reaches C1.1, U1.29 (~{RESET}/PC6)
- net RESET: now also J17.5 (Pin_5), R1.1
- no-connect marks 36 -> 37
Changed lines of the file:
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@@
   (junction (at 63.5 257.81) (diameter 0) (color 0 0 0 0)
   )
+  (junction (at 74.93 204.47) (diameter 0) (color 0 0 0 0)
+  )
   (junction (at 83.82 137.16) (diameter 0) (color 0 0 0 0)
   )
   (junction (at 40.64 92.71) (diameter 0) (color 0 0 0 0)
   )
+  (junction (at 74.93 207.01) (diameter 0) (color 0 0 0 0)
+  )
   (junction (at 63.5 265.43) (diameter 0) (color 0 0 0 0)
   )
@@
   (junction (at 26.67 252.73) (diameter 0) (color 0 0 0 0)
   )
-  (junction (at 81.28 204.47) (diameter 0) (color 0 0 0 0)
-  )
   (junction (at 227.33 213.36) (diameter 0) (color 0 0 0 0)
   )
@@
   (no_connect (at 50.8 85.09))
   (no_connect (at 35.56 171.45))
+  (no_connect (at 168.91 69.85))
   (no_connect (at 45.72 85.09))
   (no_connect (at 161.29 134.62))
@@
     (stroke (width 0) (type default))
   )
-  (wire (pts (xy 166.37 72.39) (xy 168.91 72.39))
-    (stroke (width 0) (type default))
-  )
   (wire (pts (xy 149.86 198.12) (xy 151.13 198.12))
     (stroke (width 0) (type default))
@@
     (stroke (width 0) (type default))
   )
-  (wire (pts (xy 166.37 77.47) (xy 168.91 77.47))
-    (stroke (width 0) (type default))
-  )
   (wire (pts (xy 165.1 110.49) (xy 168.91 110.49))
     (stroke (width 0) (type default))
@@
     (stroke (width 0) (type default))
   )
+  (wire (pts (xy 74.93 209.55) (xy 74.93 207.01))
+    (stroke (width 0) (type default))
+  )
   (wire (pts (xy 248.92 190.5) (xy 247.65 190.5))
     (stroke (width 0) (type default))
   )
-  (wire (pts (xy 166.37 69.85) (xy 168.91 69.85))
+  (wire (pts (xy 166.37 67.31) (xy 168.91 67.31))
     (stroke (width 0) (type default))
   )
@@
     (stroke (width 0) (type default))
   )
+  (wire (pts (xy 74.93 204.47) (xy 76.2 204.47))
+    (stroke (width 0) (type default))
+  )
   (wire (pts (xy 147.32 34.29) (xy 147.32 40.64))
     (stroke (width 0) (type default))
@@
     (stroke (width 0) (type default))
   )
+  (wire (pts (xy 81.28 207.01) (xy 74.93 207.01))
+    (stroke (width 0) (type default))
+  )
   (wire (pts (xy 226.06 237.49) (xy 248.92 237.49))
     (stroke (width 0) (type default))
@@
     (stroke (width 0) (type default))
   )
-  (wire (pts (xy 66.04 204.47) (xy 76.2 204.47))
+  (wire (pts (xy 66.04 204.47) (xy 74.93 204.47))
     (stroke (width 0) (type default))
   )
@@
     (stroke (width 0) (type default))
   )
+  (wire (pts (xy 74.93 207.01) (xy 74.93 204.47))
+    (stroke (width 0) (type default))
+  )
   (wire (pts (xy 25.4 69.85) (xy 27.94 69.85))
     (stroke (width 0) (type default))
@@
     (stroke (width 0) (type default))
   )
+  (wire (pts (xy 166.37 74.93) (xy 168.91 74.93))
+    (stroke (width 0) (type default))
+  )
   (wire (pts (xy 231.14 171.45) (xy 231.14 173.99))
     (stroke (width 0) (type default))
@@
     (stroke (width 0) (type default))
   )
-  (wire (pts (xy 81.28 204.47) (xy 81.28 207.01))
-    (stroke (width 0) (type default))
-  )
   (wire (pts (xy 165.1 171.45) (xy 168.91 171.45))
     (stroke (width 0) (type default))
@@
     (stroke (width 0) (type default))
   )
+  (wire (pts (xy 166.37 72.39) (xy 168.91 72.39))
+    (stroke (width 0) (type default))
+  )
   (wire (pts (xy 161.29 149.86) (xy 158.75 149.86))
     (stroke (width 0) (type default))
@@
     (stroke (width 0) (type default))
   )
+  (wire (pts (xy 166.37 80.01) (xy 168.91 80.01))
+    (stroke (width 0) (type default))
+  )
   (wire (pts (xy 115.57 34.29) (xy 115.57 40.64))
     (stroke (width 0) (type default))
@@
     (stroke (width 0) (type default))
   )
-  (wire (pts (xy 66.04 166.37) (xy 68.58 166.37))
+  (wire (pts (xy 166.37 77.47) (xy 168.91 77.47))
     (stroke (width 0) (type default))
   )
-  (wire (pts (xy 166.37 80.01) (xy 168.91 80.01))
+  (wire (pts (xy 66.04 166.37) (xy 68.58 166.37))
     (stroke (width 0) (type default))
   )
@@
     (stroke (width 0) (type default))
   )
-  (wire (pts (xy 81.28 204.47) (xy 83.82 204.47))
+  (wire (pts (xy 81.28 204.47) (xy 91.44 204.47))
     (stroke (width 0) (type default))
   )
@@
     (stroke (width 0) (type default))
   )
+  (wire (pts (xy 91.44 209.55) (xy 74.93 209.55))
+    (stroke (width 0) (type default))
+  )
   (wire (pts (xy 189.23 34.29) (xy 189.23 40.64))
     (stroke (width 0) (type default))
@@
     (stroke (width 0) (type default))
   )
-  (wire (pts (xy 166.37 74.93) (xy 168.91 74.93))
-    (stroke (width 0) (type default))
-  )
   (wire (pts (xy 87.63 177.8) (xy 95.25 177.8))
     (stroke (width 0) (type default))
@@
     )
   )
-  (global_label "DTR" (shape input) (at 161.29 95.25 180) (fields_autoplaced)
+  (global_label "RESET" (shape input) (at 161.29 95.25 180) (fields_autoplaced)
     (effects (font (size 1.27 1.27)) (justify right))
-    (property "Intersheetrefs" "${INTERSHEET_REFS}" (at 155.3693 95.1706 0)
+    (property "Intersheetrefs" "${INTERSHEET_REFS}" (at 152.5597 95.25 0)
       (effects (font (size 1.27 1.27)) (justify right) hide)
     )
@@
     )
   )
-  (global_label "DTR" (shape input) (at 83.82 204.47 0) (fields_autoplaced)
+  (global_label "DTR" (shape input) (at 91.44 204.47 0) (fields_autoplaced)
     (effects (font (size 1.27 1.27)) (justify left))
-    (property "Intersheetrefs" "${INTERSHEET_REFS}" (at 89.7407 204.3906 0)
+    (property "Intersheetrefs" "${INTERSHEET_REFS}" (at 97.3607 204.3906 0)
       (effects (font (size 1.27 1.27)) (justify left) hide)
     )
@@
     )
   )
+  (global_label "RESET" (shape input) (at 91.44 209.55 0) (fields_autoplaced)
+    (effects (font (size 1.27 1.27)) (justify left))
+    (property "Intersheetrefs" "${INTERSHEET_REFS}" (at 100.1703 209.55 0)
+      (effects (font (size 1.27 1.27)) (justify left) hide)
+    )
+  )
   (global_label "Column 3" (shape input) (at 71.12 31.75 0) (fields_autoplaced)
     (effects (font (size 1.27 1.27)) (justify left))
@@
     )
   )
-  (global_label "RX" (shape input) (at 166.37 72.39 180) (fields_autoplaced)
+  (global_label "RX" (shape input) (at 166.37 77.47 180) (fields_autoplaced)
     (effects (font (size 1.27 1.27)) (justify right))
-    (property "Intersheetrefs" "${INTERSHEET_REFS}" (at 161.4774 72.3106 0)
+    (property "Intersheetrefs" "${INTERSHEET_REFS}" (at 161.4774 77.3906 0)
       (effects (font (size 1.27 1.27)) (justify right) hide)
     )
@@
     )
   )
-  (global_label "+5V" (shape input) (at 166.37 80.01 180) (fields_autoplaced)
+  (global_label "+5V" (shape input) (at 166.37 72.39 180) (fields_autoplaced)
     (effects (font (size 1.27 1.27)) (justify right))
-    (property "Intersheetrefs" "${INTERSHEET_REFS}" (at 160.0864 79.9306 0)
+    (property "Intersheetrefs" "${INTERSHEET_REFS}" (at 160.0864 72.3106 0)
       (effects (font (size 1.27 1.27)) (justify right) hide)
     )
@@
     )
   )
-  (global_label "GND" (shape input) (at 166.37 69.85 180) (fields_autoplaced)
+  (global_label "GND" (shape input) (at 166.37 67.31 180) (fields_autoplaced)
     (effects (font (size 1.27 1.27)) (justify right))
-    (property "Intersheetrefs" "${INTERSHEET_REFS}" (at 160.0864 69.7706 0)
+    (property "Intersheetrefs" "${INTERSHEET_REFS}" (at 160.0864 67.2306 0)
       (effects (font (size 1.27 1.27)) (justify right) hide)
     )
@@
     )
   )
-  (global_label "DTR" (shape input) (at 166.37 77.47 180) (fields_autoplaced)
+  (global_label "DTR" (shape input) (at 166.37 80.01 180) (fields_autoplaced)
     (effects (font (size 1.27 1.27)) (justify right))
-    (property "Intersheetrefs" "${INTERSHEET_REFS}" (at 160.4493 77.3906 0)
+    (property "Intersheetrefs" "${INTERSHEET_REFS}" (at 160.4493 79.9306 0)
       (effects (font (size 1.27 1.27)) (justify right) hide)
     )
@@
     )
   )
+  (symbol (lib_id "Connector:Conn_01x06_Pin") (at 173.99 74.93 180) (unit 1)
+    (in_bom yes) (on_board yes) (dnp no) (fields_autoplaced)
+    (property "Reference" "J18" (at 175.26 72.39 0)
+      (effects (font (size 1.27 1.27)) (justify right))
+    )
+    (property "Value" "Serial Program" (at 175.26 74.93 0)
+      (effects (font (size 1.27 1.27)) (justify right))
+    )
+    (property "Footprint" "Connector_PinHeader_2.54mm:PinHeader_1x06_P2.54mm_Vertical" (at 173.99 74.93 0)
+      (effects (font (size 1.27 1.27)) hide)
+    )
+    (property "Datasheet" "~" (at 173.99 74.93 0)
+      (effects (font (size 1.27 1.27)) hide)
+    )
+    (pin "1")
+    (pin "2")
+    (pin "3")
+    (pin "4")
+    (pin "5")
+    (pin "6")
+    (instances
+      (project "RPi Arcade Hat V0-3"
+        (path "/ad210fca-1647-45d3-94e3-209006df452e"
+          (reference "J18") (unit 1)
+        )
+      )
+    )
+  )
   (symbol (lib_id "Device:R") (at 232.41 78.74 270) (unit 1)
     (in_bom yes) (on_board yes) (dnp no)
@@
         )
       )
-    )
-  )
-  (symbol (lib_id "Connector:Conn_01x05_Male") (at 173.99 74.93 180) (unit 1)
-    (in_bom yes) (on_board yes) (dnp no) (fields_autoplaced)
-    (property "Reference" "J18" (at 175.26 73.6599 0)
-      (effects (font (size 1.27 1.27)) (justify right))
-    )
-    (property "Value" "Program MCU" (at 175.26 76.1999 0)
-      (effects (font (size 1.27 1.27)) (justify right))
-    )
-    (property "Footprint" "Connector_PinHeader_2.54mm:PinHeader_1x05_P2.54mm_Vertical" (at 173.99 74.93 0)
-      (effects (font (size 1.27 1.27)) hide)
-    )
-    (property "Datasheet" "~" (at 173.99 74.93 0)
-      (effects (font (size 1.27 1.27)) hide)
-    )
-    (pin "1")
-    (pin "2")
-    (pin "3")
-    (pin "4")
-    (pin "5")
-    (instances
-      (project "RPi Arcade Hat V0-3"
-        (path "/ad210fca-1647-45d3-94e3-209006df452e"
-          (reference "J18") (unit 1)
-        )
-      )

Commit message: Changes made after testing
Parts:
- removed D1, D2, D3, D4: 1N4448W, Diode_SMD:D_SOD-123, symbol Diode:1N4448W
- removed R9: 12k, Resistor_SMD:R_1206_3216Metric, symbol Device:R
- C6, C7, C8, C9: value 100nF -> 300nF
Connections:
- net GND: now also Y1.2, Y1.4
- net MECH (12V): now also R51.2, R8.2
- net P1CRDBUTT: now also R7.1
- net P2CRDBUTT: now also R6.1
- net P3CRDBUTT: now also R5.1
- net P4CRDBUTT: now also R4.1
- no-connect marks 37 -> 35
Other:
- moved on the sheet: R51, R52, R8

Commit message: Fixed Input Matrix
Parts:
- added D1, D10, D11, D12, D13, D14, D15, D16, D17, D18, D19, D2, D20, D21, D22, D23, D24, D25, D26, D27, D28, D29, D3, D30, D31, D32, D33, D34, D35, D36, D37, D38, D39, D4, D40, D41, D6, D7, D8, D9: 1N4448W, Diode_SMD:D_SOD-123, symbol Diode:1N4448W
Connections:
- net Column 1: now also D1.2 (A), D10.2 (A), D18.2 (A), D26.2 (A), D34.2 (A); no longer J2.1 (Pin_1), J3.1 (Pin_1), J4.1 (Pin_1), J5.1 (Pin_1), J6.1 (Pin_1)
- net Column 2: now also D11.2 (A), D19.2 (A), D2.2 (A), D27.2 (A), D35.2 (A); no longer J2.2 (Pin_2), J3.2 (Pin_2), J4.2 (Pin_2), J5.2 (Pin_2), J6.2 (Pin_2)
- net Column 3: now also D12.2 (A), D20.2 (A), D28.2 (A), D3.2 (A), D36.2 (A); no longer J2.3 (Pin_3), J3.3 (Pin_3), J4.3 (Pin_3), J5.3 (Pin_3), J6.3 (Pin_3)
- net Column 4: now also D13.2 (A), D21.2 (A), D29.2 (A), D37.2 (A), D4.2 (A); no longer J2.4 (Pin_4), J3.4 (Pin_4), J4.4 (Pin_4), J5.4 (Pin_4), J6.4 (Pin_4)
- net Column 5: now also D14.2 (A), D22.2 (A), D30.2 (A), D38.2 (A), D6.2 (A); no longer J2.5 (Pin_5), J3.5 (Pin_5), J4.5 (Pin_5), J5.5 (Pin_5), J6.5 (Pin_5)
- net Column 6: now also D15.2 (A), D23.2 (A), D31.2 (A), D39.2 (A), D7.2 (A); no longer J2.6 (Pin_6), J3.6 (Pin_6), J4.6 (Pin_6), J5.6 (Pin_6), J6.6 (Pin_6)
- net Column 7: now also D16.2 (A), D24.2 (A), D32.2 (A), D40.2 (A), D8.2 (A); no longer J2.7 (Pin_7), J3.7 (Pin_7), J4.7 (Pin_7), J5.7 (Pin_7), J6.7 (Pin_7)
- net Column 8: now also D17.2 (A), D25.2 (A), D33.2 (A), D41.2 (A), D9.2 (A); no longer J2.8 (Pin_8), J3.8 (Pin_8), J4.8 (Pin_8), J5.8 (Pin_8), J6.8 (Pin_8)
- new net: D40.1 (K), J4.7 (Pin_7)
- new net: D39.1 (K), J4.6 (Pin_6)
- new net: D37.1 (K), J4.4 (Pin_4)
- new net: D34.1 (K), J4.1 (Pin_1)
- new net: D26.1 (K), J6.1 (Pin_1)
- new net: D24.1 (K), J5.7 (Pin_7)
- new net: D12.1 (K), J3.3 (Pin_3)
- new net: D6.1 (K), J2.5 (Pin_5)
- new net: D33.1 (K), J6.8 (Pin_8)
- new net: D31.1 (K), J6.6 (Pin_6)
- new net: D14.1 (K), J3.5 (Pin_5)
- new net: D3.1 (K), J2.3 (Pin_3)
- new net: D2.1 (K), J2.2 (Pin_2)
- new net: D25.1 (K), J5.8 (Pin_8)
- new net: D36.1 (K), J4.3 (Pin_3)
- new net: D35.1 (K), J4.2 (Pin_2)
- new net: D38.1 (K), J4.5 (Pin_5)
- new net: D41.1 (K), J4.8 (Pin_8)
- new net: D9.1 (K), J2.8 (Pin_8)
- new net: D27.1 (K), J6.2 (Pin_2)
- new net: D28.1 (K), J6.3 (Pin_3)
- new net: D29.1 (K), J6.4 (Pin_4)
- new net: D30.1 (K), J6.5 (Pin_5)
- new net: D32.1 (K), J6.7 (Pin_7)
- new net: D19.1 (K), J5.2 (Pin_2)
- new net: D13.1 (K), J3.4 (Pin_4)
- new net: D1.1 (K), J2.1 (Pin_1)
- new net: D4.1 (K), J2.4 (Pin_4)
- new net: D10.1 (K), J3.1 (Pin_1)
- new net: D11.1 (K), J3.2 (Pin_2)
- new net: D15.1 (K), J3.6 (Pin_6)
- new net: D16.1 (K), J3.7 (Pin_7)
- new net: D17.1 (K), J3.8 (Pin_8)
- new net: D7.1 (K), J2.6 (Pin_6)
- new net: D8.1 (K), J2.7 (Pin_7)
- new net: D18.1 (K), J5.1 (Pin_1)
- new net: D20.1 (K), J5.3 (Pin_3)
- new net: D21.1 (K), J5.4 (Pin_4)
- new net: D22.1 (K), J5.5 (Pin_5)
- new net: D23.1 (K), J5.6 (Pin_6)
Other:
- moved on the sheet: J4

Commit message: Additional Fixes
Parts:
- added D42, D43, D44, D45: 1N4448W, Diode_SMD:D_SOD-123, symbol Diode:1N4448W
- added R17, R18, R19, R20, R9: 10k, Resistor_SMD:R_1206_3216Metric, symbol Device:R
Connections:
- net Column 9: now also D42.2 (A), D43.2 (A), D44.2 (A), D45.2 (A); no longer Q4.3 (C), Q5.3 (C), Q6.3 (C), Q7.3 (C)
- net GND: now also R17.1, R18.1, R19.1, R20.1, R9.1
- net Row 1: now also R9.2
- net Row 2: now also R17.2
- net Row 3: now also R18.2
- net Row 4: now also R19.2
- net Row 5: now also R20.2
- new net: D45.1 (K), Q4.3 (C)
- new net: D44.1 (K), Q5.3 (C)
- new net: D42.1 (K), Q7.3 (C)
- new net: D43.1 (K), Q6.3 (C)

Commit message: fixes and updates
Parts:
- removed Q5, Q6, Q7: BC847, Package_TO_SOT_SMD:SOT-23, symbol Transistor_BJT:BC847
- added Q1, Q2, Q3: BC847, Package_TO_SOT_SMD:SOT-23, symbol Transistor_BJT:BC847
- added R21, R22, R23, R24: 10k, Resistor_SMD:R_1206_3216Metric, symbol Device:R
- added RLY1, RLY2, RLY3, RLY4: 9007-05-00, digikey-footprints:Relay_Reed_9007-05-00, symbol dk_Reed-Relays:9007-05-00
- J8: footprint Connector_PinHeader_2.54mm:PinHeader_1x02_P2.54mm_Vertical -> 2 Way Terminal Block:CONN_1890963_PXC
Connections:
- net +5V: now also Q4.3 (C), Q1.3 (C), Q2.3 (C), Q3.3 (C)
- net GND: now also R21.2, R22.2, R23.2, R24.2, RLY1.3, RLY2.3, RLY3.3, RLY4.3; no longer J1.9 (GND)
- net Row 1: now also RLY1.4; no longer Q4.2 (E)
- net Row 2: now also RLY2.4
- net Row 3: now also RLY3.4
- net Row 4: now also RLY4.4
- net at R36.1: now also Q1.1 (B)
- net at R38.1: now also Q3.1 (B)
- net at D45.1 (K): now also RLY1.1; no longer Q4.3 (C)
- net at D44.1 (K): now also RLY2.1
- net at D42.1 (K): now also RLY4.1
- net at R37.1: now also Q2.1 (B)
- net at D43.1 (K): now also RLY3.1
- new net: Q1.2 (E), R21.1, RLY4.2
- new net: Q4.2 (E), R24.1, RLY1.2
- new net: Q3.2 (E), R23.1, RLY2.2
- new net: Q2.2 (E), R22.1, RLY3.2
- no-connect marks 35 -> 36
Other:
- moved on the sheet: C6, C7, C8, C9, J13, J14, J15, J16, R10, R11, R12, R13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
